File: schematic/motion_wheels/motion_wheels.kicad_sch (KiCad schematic)
At the start: 7 parts, among them J1 Conn_ZKP_1.3, M1 Motor_DC, M2 Motor_DC, U1 L9110S, U2 ESP32_DEVKITV1_36PINS, U3 GY-91, U5 LED_MODULE_RG

Commit message: Update schematic
Parts:
- removed J1: Conn_ZKP_1.3, symbol zk_connectors:Conn_ZKP_1.3
- added U4: HW-021_TJA1050, symbol zk_modules:HW-021_TJA1050
Connections:
- net SCL is gone; now on an unnamed net: U2.10 (IO27)
- net SDA is gone; now on an unnamed net: U2.11 (IO14)
- net at U2.12 (IO12): now also U1.5 (A1_IN)
- net at U2.13 (IO13): now also U1.6 (A2_IN)
- net GNDD: now reaches U2.17 (GND)
- net GNDD: now also U3.3 (GND), U5.3 (GND), U4.4 (GND)
- net +5VDD: now reaches U2.18 (VIN)
- net +5VDD: now also U3.1 (VIN), U4.1 (VCC)
- net at U2.19 (IO23): no longer U5.1 (RED)
- net at U2.20 (IO22/SCL): no longer U5.2 (GREEN)
- net at U2.23 (IO21/SDA): no longer U3.5 (SDA)
- net at U2.24 (IO19): no longer U3.4 (SCL)
- net at U2.25 (IO18): now also U3.5 (SDA)
- net at U2.26 (IO5): now also U3.4 (SCL)
- net at U2.27 (IO17/TXD2): now also U5.1 (RED)
- net at U2.28 (IO16/RXD2): now also U5.2 (GREEN)
- net at U1.1 (B1_IN): no longer U2.6 (IO32)
- net at U1.2 (B2_IN): no longer U2.7 (IO33)
- net at U2.8 (IO25): now also U4.2 (TX); no longer U1.5 (A1_IN)
- net at U2.9 (IO26): now also U4.3 (RX); no longer U1.6 (A2_IN)
- net 5V_HI_I renamed +5V_MTR
- net 5V_LO_I: no longer names the net of U2.38 (USB_VIN)
- net 5V_LO_I: no longer U3.1 (VIN)
- net GND_HI_I renamed GND
- removed net GND_LO_I: U2.37 (USB_GND), U3.3 (GND), U5.3 (GND)
Other:
- removed sheet Power
- moved on the sheet: M1, M2, U1, U3, U5
